File: Zolotarev.kicad_pcb (KiCad board)
At the start: 2 copper layers, 185 x 185 mm, 176 parts, among them J1 RF_IN, J2 RF_OUT, J3 Conn_02x05_Odd_Even, K1 G5LE-1, K10 G5LE-1, K11 G5LE-1, K12 G5LE-1, K13 G5LE-1, K14 G5LE-1, K2 G5LE-1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

Commit message: 3 bands over 7
Parts:
- moved C205 292.5 mm to (77.0, 76.0), turned to 90 degrees
- moved C37 251.9 mm to (99.5, 61.5), turned to 90 degrees
- moved C36 245.7 mm to (103.5, 61.5), turned to 90 degrees
- moved C25 242.4 mm to (119.8, 61.5), turned to -90 degrees
- moved C22 242.2 mm to (85.8, 62.8), turned to 90 degrees
- moved C35 239.4 mm to (107.5, 61.5), turned to 90 degrees
- moved C24 239.2 mm to (115.8, 61.5), turned to -90 degrees
- moved C26 237.6 mm to (152.8, 61.5), turned to -90 degrees
- moved C23 236.1 mm to (111.7, 61.5), turned to -90 degrees
- moved C21 234.9 mm to (89.8, 63.8), turned to 90 degrees
- moved C20 227.9 mm to (93.8, 64.5), turned to 90 degrees
- moved C224 224.7 mm to (197.0, 73.0), turned to -90 degrees
- moved C225 221.7 mm to (195.0, 54.9), turned to 90 degrees
- moved C222 220.4 mm to (197.0, 96.0), turned to -90 degrees
- moved C223 216.9 mm to (195.0, 77.0), turned to 90 degrees
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Connections:
- D3 pad 2: unconnected-(D3-A-Pad2) -> 60+40m
Routing:
- net 60+40m: track 0.00 -> 150.8 mm
- net 80m: track 0.00 -> 145.7 mm
- net +12V: track 180.7 -> 289.0 mm
- net Net-(C26-Pad1): track 0.00 -> 54.9 mm
- net Net-(C46-Pad1): track 0.00 -> 48.4 mm
- net Net-(C30-Pad1): track 0.00 -> 47.9 mm
- net Net-(C23-Pad1): track 0.00 -> 45.6 mm
- net Net-(C38-Pad1): track 0.00 -> 44.7 mm
- net Net-(C38-Pad2): track 0.00 -> 43.7 mm
- net Net-(C50-Pad1): track 0.00 -> 41.7 mm
- net Net-(C20-Pad1): track 0.00 -> 38.7 mm
- net 160m: track 146.5 -> 145.8 mm
- net GND: vias 212 -> 655

Commit message: 5 bands routed, 2 more to come
Parts:
- moved D8 258.9 mm to (223.0, 180.0)
- moved D6 252.8 mm to (221.5, 156.5)
- moved C216 246.9 mm to (202.5, 155.0)
- moved C217 246.9 mm to (202.5, 158.0)
- moved C214 246.2 mm to (204.0, 178.5)
- moved C215 246.2 mm to (204.0, 181.5)
- moved C218 234.7 mm to (197.2, 142.0), turned to -90 degrees
- moved C220 225.5 mm to (197.0, 118.5), turned to -90 degrees
- moved C219 225.5 mm to (195.0, 122.8), turned to 90 degrees
- moved C221 219.3 mm to (195.0, 100.0), turned to 90 degrees
- moved D11 217.6 mm to (199.5, 109.0), turned to -90 degrees
- moved D10 204.3 mm to (199.5, 132.2), turned to -90 degrees
- moved C61 188.1 mm to (147.6, 108.2), turned to -90 degrees
- moved C59 185.4 mm to (119.5, 108.8), turned to -90 degrees
- moved C60 184.2 mm to (142.5, 108.2), turned to -90 degrees
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Connections:
- D4 pad 1: unconnected-(D4-K-Pad1) -> +12V
- D5 pad 1: unconnected-(D5-K-Pad1) -> +12V
Routing:
- net 17+15m: track 0.00 -> 145.8 mm
- net 30+20m: track 0.00 -> 145.3 mm
- net +12V: track 289.0 -> 420.0 mm
- net RF_IN: track 29.1 -> 150.6 mm
- net RF_OUT: track 26.4 -> 138.4 mm
- net Net-(C69-Pad1): track 0.00 -> 53.6 mm
- net Net-(C56-Pad1): track 0.00 -> 50.9 mm
- net Net-(C60-Pad1): track 0.00 -> 48.5 mm
- net Net-(C65-Pad1): track 0.00 -> 41.9 mm
- net Net-(C67-Pad1): track 0.00 -> 41.1 mm
- net Net-(C62-Pad1): track 0.00 -> 40.7 mm
- net Net-(C71-Pad1): track 0.00 -> 40.5 mm
- net Net-(C53-Pad1): track 0.00 -> 30.8 mm
- net GND: vias 655 -> 1045
