File: Zolotarev.kicad_pcb (KiCad board)
At the start: 2 copper layers, 185 x 185 mm, 174 parts, among them J1 RF_IN, J2 RF_OUT, J3 Conn_02x05_Odd_Even, K1 G5LE-1, K10 G5LE-1, K11 G5LE-1, K12 G5LE-1, K13 G5LE-1, K14 G5LE-1, K2 G5LE-1, K3 G5LE-1, K4 G5LE-1, K5 G5LE-1, K6 G5LE-1, K7 G5LE-1, K8 G5LE-1, K9 G5LE-1

Commit message: control connector and some ferrites later
Parts:
- removed REF**: KiCad-Logo2_5mm_SilkScreen, Symbol:KiCad-Logo2_5mm_SilkScreen
- removed REF**: OSHW-Logo2_9.8x8mm_SilkScreen, Symbol:OSHW-Logo2_9.8x8mm_SilkScreen
- added FB10: FB, Inductor_SMD:L_0805_2012Metric_Pad1.15x1.40mm_HandSolder, F.Cu at (-36.2, 13.4)
- added FB11: FB, Inductor_SMD:L_0805_2012Metric_Pad1.15x1.40mm_HandSolder, F.Cu at (-36.2, 16.4)
- added FB12: FB, Inductor_SMD:L_0805_2012Metric_Pad1.15x1.40mm_HandSolder, F.Cu at (-36.2, 19.4)
- added FB13: FB, Inductor_SMD:L_0805_2012Metric_Pad1.15x1.40mm_HandSolder, F.Cu at (-36.2, 22.3)
- added FB14: FB, Inductor_SMD:L_0805_2012Metric_Pad1.15x1.40mm_HandSolder, F.Cu at (-36.2, 25.2)
- added FB15: FB, Inductor_SMD:L_0805_2012Metric_Pad1.15x1.40mm_HandSolder, F.Cu at (-36.2, 28.2)
- added FB16: FB, Inductor_SMD:L_0805_2012Metric_Pad1.15x1.40mm_HandSolder, F.Cu at (-36.2, 31.1)
- added FB17: FB, Inductor_SMD:L_0805_2012Metric_Pad1.15x1.40mm_HandSolder, F.Cu at (-36.2, 34.1)
- added FB18: FB, Inductor_SMD:L_0805_2012Metric_Pad1.15x1.40mm_HandSolder, F.Cu at (-31.5, 13.4)
- added FB19: FB, Inductor_SMD:L_0805_2012Metric_Pad1.15x1.40mm_HandSolder, F.Cu at (-31.5, 16.4)
- added FB2: FB, Inductor_SMD:L_0805_2012Metric_Pad1.15x1.40mm_HandSolder, B.Cu at (218.8, 65.8)
- added FB20: FB, Inductor_SMD:L_0805_2012Metric_Pad1.15x1.40mm_HandSolder, F.Cu at (-31.5, 19.4)
- added FB21: FB, Inductor_SMD:L_0805_2012Metric_Pad1.15x1.40mm_HandSolder, F.Cu at (-31.5, 22.3)
- added FB22: FB, Inductor_SMD:L_0805_2012Metric_Pad1.15x1.40mm_HandSolder, F.Cu at (-31.5, 25.2)
- added FB23: FB, Inductor_SMD:L_0805_2012Metric_Pad1.15x1.40mm_HandSolder, F.Cu at (-31.5, 28.2)
- added FB24: FB, Inductor_SMD:L_0805_2012Metric_Pad1.15x1.40mm_HandSolder, F.Cu at (-31.5, 31.1)
- added FB25: FB, Inductor_SMD:L_0805_2012Metric_Pad1.15x1.40mm_HandSolder, F.Cu at (-31.5, 34.1)
- added FB26: FB, Inductor_SMD:L_0805_2012Metric_Pad1.15x1.40mm_HandSolder, F.Cu at (-26.7, 13.4)
- added FB27: FB, Inductor_SMD:L_0805_2012Metric_Pad1.15x1.40mm_HandSolder, F.Cu at (-26.7, 16.4)
- added FB28: FB, Inductor_SMD:L_0805_2012Metric_Pad1.15x1.40mm_HandSolder, F.Cu at (-26.7, 19.4)
- added FB29: FB, Inductor_SMD:L_0805_2012Metric_Pad1.15x1.40mm_HandSolder, F.Cu at (-26.7, 22.3)
- added FB3: FB, Inductor_SMD:L_0805_2012Metric_Pad1.15x1.40mm_HandSolder, B.Cu at (218.0, 89.0)
- added FB30: FB, Inductor_SMD:L_0805_2012Metric_Pad1.15x1.40mm_HandSolder, F.Cu at (-26.7, 25.2)
- added FB31: FB, Inductor_SMD:L_0805_2012Metric_Pad1.15x1.40mm_HandSolder, F.Cu at (-26.7, 28.2)
- added FB32: FB, Inductor_SMD:L_0805_2012Metric_Pad1.15x1.40mm_HandSolder, F.Cu at (-26.7, 31.1)
- added FB33: FB, Inductor_SMD:L_0805_2012Metric_Pad1.15x1.40mm_HandSolder, F.Cu at (-26.7, 34.1)
- added FB34: FB, Inductor_SMD:L_0805_2012Metric_Pad1.15x1.40mm_HandSolder, F.Cu at (-22.0, 13.4)
- added FB35: FB, Inductor_SMD:L_0805_2012Metric_Pad1.15x1.40mm_HandSolder, F.Cu at (-22.0, 16.4)
- added FB36: FB, Inductor_SMD:L_0805_2012Metric_Pad1.15x1.40mm_HandSolder, F.Cu at (-22.0, 19.4)
- added FB37: FB, Inductor_SMD:L_0805_2012Metric_Pad1.15x1.40mm_HandSolder, F.Cu at (-22.0, 22.3)
- added FB38: FB, Inductor_SMD:L_0805_2012Metric_Pad1.15x1.40mm_HandSolder, F.Cu at (-22.0, 25.2)
- added FB4: FB, Inductor_SMD:L_0805_2012Metric_Pad1.15x1.40mm_HandSolder, B.Cu at (216.9, 111.1)
- added FB5: FB, Inductor_SMD:L_0805_2012Metric_Pad1.15x1.40mm_HandSolder, B.Cu at (218.1, 129.7)
- added FB6: FB, Inductor_SMD:L_0805_2012Metric_Pad1.15x1.40mm_HandSolder, B.Cu at (218.9, 152.1)
- added FB7: FB, Inductor_SMD:L_0805_2012Metric_Pad1.15x1.40mm_HandSolder, B.Cu at (220.5, 176.5)
- added FB8: FB, Inductor_SMD:L_0805_2012Metric_Pad1.15x1.40mm_HandSolder, B.Cu at (221.3, 41.3)
- added FB9: FB, Inductor_SMD:L_0805_2012Metric_Pad1.15x1.40mm_HandSolder, B.Cu at (219.3, 45.3)
- added G***: LOGO, Munin_logo:Munin, F.Cu at (161.0, 185.0)
- added G***: LOGO, Munin_logo:Munin, B.Cu at (161.0, 166.0)
Connections:
- C200 pad 1: +12V -> Net-(D1-K)
- C201 pad 1: 160m -> Net-(D1-A)
- C202 pad 1: +12V -> Net-(D2-K)
- C203 pad 1: 80m -> Net-(D2-A)
- C204 pad 1: +12V -> Net-(D3-K)
- C205 pad 1: 60+40m -> Net-(D3-A)
- C206 pad 1: +12V -> Net-(D4-K)
- C207 pad 1: 30+20m -> Net-(D4-A)
- C208 pad 1: +12V -> Net-(D5-K)
- C209 pad 1: 17+15m -> Net-(D5-A)
- C210 pad 1: +12V -> Net-(D6-K)
- C211 pad 1: 12+10m -> Net-(D6-A)
- C212 pad 1: +12V -> Net-(D7-K)
- C213 pad 1: 6m -> Net-(D7-A)
- C214 pad 1: 6m -> Net-(D8-A)
- C215 pad 1: +12V -> Net-(D8-K)
- C216 pad 1: 12+10m -> Net-(D9-A)
- C217 pad 1: +12V -> Net-(D9-K)
- C218 pad 1: 17+15m -> Net-(D10-A)
- C219 pad 1: +12V -> Net-(D10-K)
- C220 pad 1: 30+20m -> Net-(D11-A)
- C221 pad 1: +12V -> Net-(D11-K)
- C222 pad 1: 60+40m -> Net-(D12-A)
- C223 pad 1: +12V -> Net-(D12-K)
- C224 pad 1: 80m -> Net-(D13-A)
- C225 pad 1: +12V -> Net-(D13-K)
- C226 pad 1: 160m -> Net-(D14-A)
- C227 pad 1: +12V -> Net-(D14-K)
- D1 pad 1: +12V -> Net-(D1-K)
- D1 pad 2: 160m -> Net-(D1-A)
- D10 pad 1: +12V -> Net-(D10-K)
- D10 pad 2: 17+15m -> Net-(D10-A)
- D11 pad 1: +12V -> Net-(D11-K)
- D11 pad 2: 30+20m -> Net-(D11-A)
- D12 pad 1: +12V -> Net-(D12-K)
- D12 pad 2: 60+40m -> Net-(D12-A)
- D13 pad 1: +12V -> Net-(D13-K)
- D13 pad 2: 80m -> Net-(D13-A)
- D14 pad 1: +12V -> Net-(D14-K)
- D14 pad 2: 160m -> Net-(D14-A)
- D2 pad 1: +12V -> Net-(D2-K)
- D2 pad 2: 80m -> Net-(D2-A)
- D3 pad 1: +12V -> Net-(D3-K)
- D3 pad 2: 60+40m -> Net-(D3-A)
- D4 pad 1: +12V -> Net-(D4-K)
- D4 pad 2: 30+20m -> Net-(D4-A)
- D5 pad 1: +12V -> Net-(D5-K)
- D5 pad 2: 17+15m -> Net-(D5-A)
- D6 pad 1: +12V -> Net-(D6-K)
- D6 pad 2: 12+10m -> Net-(D6-A)
- D7 pad 1: +12V -> Net-(D7-K)
- D7 pad 2: 6m -> Net-(D7-A)
- D8 pad 1: +12V -> Net-(D8-K)
- D8 pad 2: 6m -> Net-(D8-A)
- D9 pad 1: +12V -> Net-(D9-K)
- D9 pad 2: 12+10m -> Net-(D9-A)
- J3 pad 1: +12V -> Net-(J3-Pin_1)
- J3 pad 10: GND -> Net-(J3-Pin_10)
- J3 pad 2: GND -> Net-(J3-Pin_2)
- J3 pad 3: 160m -> Net-(J3-Pin_3)
- J3 pad 4: 80m -> Net-(J3-Pin_4)
- J3 pad 5: 60+40m -> Net-(J3-Pin_5)
- J3 pad 6: 30+20m -> GND
- J3 pad 7: 17+15m -> Net-(J3-Pin_7)
- J3 pad 8: 12+10m -> GND
- J3 pad 9: 6m -> Net-(J3-Pin_9)
- K1 pad 2: 160m -> Net-(D1-A)
- K1 pad 5: +12V -> Net-(D1-K)
- K10 pad 2: 17+15m -> Net-(D10-A)
- K10 pad 5: +12V -> Net-(D10-K)
- K11 pad 2: 12+10m -> Net-(D6-A)
- K11 pad 5: +12V -> Net-(D6-K)
- K12 pad 2: 12+10m -> Net-(D9-A)
- K12 pad 5: +12V -> Net-(D9-K)
- K13 pad 2: 6m -> Net-(D7-A)
- K13 pad 5: +12V -> Net-(D7-K)
- K14 pad 2: 6m -> Net-(D8-A)
- K14 pad 5: +12V -> Net-(D8-K)
- K2 pad 2: 160m -> Net-(D14-A)
- K2 pad 5: +12V -> Net-(D14-K)
- K3 pad 2: 80m -> Net-(D2-A)
- K3 pad 5: +12V -> Net-(D2-K)
- K4 pad 2: 80m -> Net-(D13-A)
- K4 pad 5: +12V -> Net-(D13-K)
- K5 pad 2: 60+40m -> Net-(D3-A)
- K5 pad 5: +12V -> Net-(D3-K)
- K6 pad 2: 60+40m -> Net-(D12-A)
- K6 pad 5: +12V -> Net-(D12-K)
- K7 pad 2: 30+20m -> Net-(D4-A)
- K7 pad 5: +12V -> Net-(D4-K)
- K8 pad 2: 30+20m -> Net-(D11-A)
- K8 pad 5: +12V -> Net-(D11-K)
- K9 pad 2: 17+15m -> Net-(D5-A)
- K9 pad 5: +12V -> Net-(D5-K)
Routing:
- net Net-(J3-Pin_4): track 0.00 -> 69.4 mm
- net Net-(J3-Pin_2): track 0.00 -> 61.2 mm
- net Net-(J3-Pin_10): track 0.00 -> 60.4 mm
- net Net-(J3-Pin_1): track 0.00 -> 39.2 mm
- net Net-(J3-Pin_9): track 0.00 -> 35.6 mm
- net Net-(J3-Pin_3): track 0.00 -> 20.3 mm
- net Net-(J3-Pin_7): track 0.00 -> 16.7 mm
- net +12V: track 567.9 -> 561.5 mm
- net Net-(J3-Pin_5): track 0.00 -> 3.99 mm
- net 6m: track 165.8 -> 169.7 mm, vias 0 -> 1
- net 17+15m: track 167.8 -> 171.0 mm, vias 0 -> 1
- net 12+10m: track 167.9 -> 170.8 mm, vias 0 -> 1
- net 60+40m: track 173.7 -> 176.1 mm, vias 0 -> 1
- net 80m: track 168.2 -> 170.5 mm, vias 0 -> 1
- net 160m: track 167.4 -> 169.6 mm, vias 0 -> 1
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Other:
- board text added: "Huginn ok Muninn fljúga hverjan dag Jörmungrund yfir; óumk ek of Hugin, at hann aftr né komi-t, þó sjámk meir of Munin."

Commit message: routing, silk, zone cleanup and Gerber completed, RTM release
Parts:
- removed C1: 2.2n, ATC_B:ATC_500_HandSoldering
- removed FB25: FB, Inductor_SMD:L_0805_2012Metric_Pad1.15x1.40mm_HandSolder
- added C10b1: Adj, ATC_B:ATC_500_HandSoldering, B.Cu at (108.4, 37.8)
- added C11b1: Adj, ATC_B:ATC_500_HandSoldering, B.Cu at (116.6, 38.0)
- added C12: 2.2n, ATC_B:ATC_500_HandSoldering, B.Cu at (55.0, 46.0)
- added C12b1: Adj, ATC_B:ATC_500_HandSoldering, B.Cu at (56.6, 53.4)
- added C12c1: Adj, ATC_B:ATC_500_HandSoldering, B.Cu at (52.6, 52.2)
- added C15b1: Adj, ATC_B:ATC_500_HandSoldering, B.Cu at (126.8, 50.0)
- added C15c1: Adj, ATC_B:ATC_500_HandSoldering, B.Cu at (138.4, 50.0)
- added C19b1: Adj, ATC_B:ATC_500_HandSoldering, B.Cu at (73.0, 49.0)
- added C23b1: Adj, ATC_B:ATC_500_HandSoldering, B.Cu at (92.2, 73.4)
- added C24b1: Adj, ATC_B:ATC_500_HandSoldering, B.Cu at (92.2, 77.2)
- added C26b1: Adj, ATC_B:ATC_500_HandSoldering, B.Cu at (117.6, 61.6)
- added C26c1: Adj, ATC_B:ATC_500_HandSoldering, B.Cu at (102.6, 60.0)
- added C27b1: Adj, ATC_B:ATC_500_HandSoldering, B.Cu at (106.4, 60.0)
- added C28b1: Adj, ATC_B:ATC_500_HandSoldering, B.Cu at (121.4, 61.6)
- added C2b1: Adj, ATC_B:ATC_500_HandSoldering, B.Cu at (93.2, 53.0)
- added C40b1: Adj, ATC_B:ATC_500_HandSoldering, B.Cu at (52.2, 90.6)
- added C42b1: Adj, ATC_B:ATC_500_HandSoldering, B.Cu at (92.8, 96.6)
- added C43b1: Adj, ATC_B:ATC_500_HandSoldering, B.Cu at (92.8, 100.4)
- added C46b1: Adj, ATC_B:ATC_500_HandSoldering, B.Cu at (119.0, 90.0)
- added C46c1: Adj, ATC_B:ATC_500_HandSoldering, B.Cu at (123.0, 90.0)
- added C50b1: Adj, ATC_B:ATC_500_HandSoldering, B.Cu at (146.8, 94.0)
- added C56b1: Adj, ATC_B:ATC_500_HandSoldering, B.Cu at (94.2, 119.0)
- added C60b1: Adj, ATC_B:ATC_500_HandSoldering, B.Cu at (119.4, 113.2)
- added C69b1: Adj, ATC_B:ATC_500_HandSoldering, B.Cu at (119.4, 136.6)
- added C6b1: Adj, ATC_B:ATC_500_HandSoldering, B.Cu at (90.6, 50.4)
- added H5: M3, MountingHole:MountingHole_3.5mm_Pad_Via, F.Cu at (53.4, 212.6)
- added H6: M3, MountingHole:MountingHole_3.5mm_Pad_Via, F.Cu at (185.1, 212.5)
- added H7: M3, MountingHole:MountingHole_3.5mm_Pad_Via, F.Cu at (157.4, 212.5)
- added H8: M3, MountingHole:MountingHole_3.5mm_Pad_Via, F.Cu at (25.9, 212.6)
- FB10, FB11, FB12, FB13, FB14, FB15, FB16, FB17, FB18, FB19, FB20, FB21, FB22, FB23, FB24, FB26, FB27, FB28, FB29, FB30, FB31, FB32, FB33, FB34, FB35, FB36, FB37, FB38: moved to B.Cu
- moved FB11 262.6 mm to (160.8, 190.0)
- moved FB32 243.4 mm to (167.8, 177.4), turned to -135 degrees
- moved FB15 242.8 mm to (161.2, 169.5), turned to 45 degrees
- moved FB14 231.8 mm to (161.4, 146.4), turned to 45 degrees
- moved FB33 228.5 mm to (167.8, 154.0), turned to -135 degrees
- moved FB34 221.6 mm to (167.2, 128.8), turned to -135 degrees
- moved FB16 218.2 mm to (161.7, 122.9), turned to 45 degrees
- moved FB18 211.4 mm to (161.3, 100.1), turned to 45 degrees
- moved FB35 209.1 mm to (167.0, 105.8), turned to -135 degrees
- moved FB23 199.1 mm to (161.6, 76.8), turned to 45 degrees
- moved FB36 199.1 mm to (166.8, 82.6), turned to -135 degrees
- moved FB22 196.0 mm to (162.1, 55.9), turned to 45 degrees
- moved FB37 192.7 mm to (167.1, 59.7), turned to -135 degrees
- moved FB38 190.0 mm to (167.6, 38.6), turned to -135 degrees
- moved FB10 181.5 mm to (47.6, 174.4), turned to 45 degrees
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Connections:
- C214 pad 1: Net-(D8-A) -> 6m
- C216 pad 1: Net-(D9-A) -> 12+10m
- C218 pad 1: Net-(D10-A) -> 17+15m
- C220 pad 1: Net-(D11-A) -> 30+20m
- C222 pad 1: Net-(D12-A) -> 60+40m
- C224 pad 1: Net-(D13-A) -> 80m
- C226 pad 1: Net-(D14-A) -> 160m
- D10 pad 2: Net-(D10-A) -> 17+15m
- D11 pad 2: Net-(D11-A) -> 30+20m
- D12 pad 2: Net-(D12-A) -> 60+40m
- D13 pad 2: Net-(D13-A) -> 80m
- D14 pad 2: Net-(D14-A) -> 160m
- D8 pad 2: Net-(D8-A) -> 6m
- D9 pad 2: Net-(D9-A) -> 12+10m
- FB10 pad 2: 6m -> Net-(FB10-Pad2)
- FB11 pad 1: 6m -> Net-(FB10-Pad2)
- FB11 pad 2: Net-(D8-A) -> 6m
- FB12 pad 2: 12+10m -> Net-(FB12-Pad2)
- FB13 pad 2: 17+15m -> Net-(FB13-Pad2)
- FB14 pad 1: 17+15m -> Net-(FB13-Pad2)
- FB14 pad 2: Net-(D10-A) -> 17+15m
- FB15 pad 1: 12+10m -> Net-(FB12-Pad2)
- FB15 pad 2: Net-(D9-A) -> 12+10m
- FB16 pad 1: 30+20m -> Net-(FB16-Pad1)
- FB16 pad 2: Net-(D11-A) -> 30+20m
- FB17 pad 2: 30+20m -> Net-(FB16-Pad1)
- FB18 pad 1: 60+40m -> Net-(FB18-Pad1)
- FB18 pad 2: Net-(D12-A) -> 60+40m
- FB19 pad 2: 60+40m -> Net-(FB18-Pad1)
- FB20 pad 2: 80m -> Net-(FB20-Pad2)
- FB21 pad 2: 160m -> Net-(FB21-Pad2)
- FB22 pad 1: 160m -> Net-(FB21-Pad2)
- FB22 pad 2: Net-(D14-A) -> 160m
- FB23 pad 1: 80m -> Net-(FB20-Pad2)
- FB23 pad 2: Net-(D13-A) -> 80m
- K10 pad 2: Net-(D10-A) -> 17+15m
- K12 pad 2: Net-(D9-A) -> 12+10m
- K14 pad 2: Net-(D8-A) -> 6m
- K2 pad 2: Net-(D14-A) -> 160m
- K4 pad 2: Net-(D13-A) -> 80m
- K6 pad 2: Net-(D12-A) -> 60+40m
- K8 pad 2: Net-(D11-A) -> 30+20m
Routing:
- net 60+40m: track 176.1 -> 35.0 mm
- net 30+20m: track 167.7 -> 31.3 mm
- net 80m: track 170.5 -> 34.1 mm
- net 17+15m: track 171.0 -> 34.7 mm
- net 12+10m: track 170.8 -> 34.8 mm
- net 160m: track 169.6 -> 34.1 mm
- net 6m: track 169.7 -> 36.7 mm
- net Net-(FB18-Pad1): track 0.00 -> 126.6 mm
- net Net-(FB21-Pad2): track 0.00 -> 123.1 mm
- net Net-(FB16-Pad1): track 0.00 -> 122.6 mm
- net Net-(FB20-Pad2): track 0.00 -> 122.6 mm
- net Net-(FB13-Pad2): track 0.00 -> 122.2 mm
- net Net-(FB12-Pad2): track 0.00 -> 122.1 mm
- net Net-(FB10-Pad2): track 0.00 -> 119.9 mm
- net Net-(J3-Pin_4): track 69.4 -> 8.64 mm
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Other:
- board size 185 x 185 mm -> 190 x 200 mm
- board text added: "Hugin and Munin fly every day Across the vast earth; {dblquote}I fear for Hugin that he will not return; But I fear even more for Munin{dblquote}"
